File: eirini.kicad_pcb (KiCad board)
At the start: 2 copper layers, 142.2 x 127 mm, 14 parts, among them U2 ESP32-C3_SUPERMINI

Commit message: Change text
Other:
- board text added: "Brno 2024"
- board text removed: "Ειρήνη-Board"
- board text removed: "Σε ευχαριστώ για όλα! Ti voglio bene"
Changed lines of the file:
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@@
 		(layer "Edge.Cuts")
 	)
-	(gr_text "Ειρήνη-Board"
-		(at 92.71 76.2 0)
+	(gr_text "Brno 2024"
+		(at 103.5 75 0)
 		(layer "B.SilkS")
 		(effects
 			(font
-				(size 1.5 1.5)
+				(face "Vafle VUT")
+				(size 5.5 5.5)
 				(thickness 0.3)
 				(bold yes)
@@
 			(justify left bottom mirror)
 		)
-	)
-	(gr_text "Σε ευχαριστώ για όλα!\n  Ti voglio bene"
-		(at 91.44 80.01 0)
-		(layer "B.SilkS")
-		(effects
-			(font
-				(size 0.8 0.8)
-				(thickness 0.15)
-				(bold yes)
+		(render_cache "Brno 2024" 0
+			(polygon
+				(pts
+					(xy 103.115806 74.065) (xy 100.458688 74.065) (xy 100.179156 74.040662) (xy 99.867387 73.945178)
+					(xy 99.603504 73.783257) (xy 99.393992 73.561171) (xy 99.245341 73.285193) (xy 99.164036 72.961595)
+					(xy 99.150279 72.747187) (xy 99.150279 72.435533) (xy 99.170547 72.189703) (xy 100.305547 72.189703)
+					(xy 100.305547 72.674647) (xy 100.400756 72.935086) (xy 100.652128 73.033318) (xy 101.960537 73.033318)
+					(xy 101.960537 71.831032) (xy 100.652128 71.831032) (xy 100.400756 71.929264) (xy 100.305547 72.189703)
+					(xy 99.170547 72.189703) (xy 99.173293 72.156394) (xy 99.255553 71.863703) (xy 99.392906 71.611822)
+					(xy 99.580542 71.406319) (xy 99.74269 71.291011) (xy 99.74269 71.260115) (xy 99.541798 71.062329)
+					(xy 99.391911 70.819333) (xy 99.298192 70.536791) (xy 99.266323 70.261584) (xy 99.265806 70.220373)
+					(xy 99.265806 70.022903) (xy 100.421074 70.022903) (xy 100.421074 70.4568) (xy 100.52775 70.715351)
+					(xy 100.766311 70.798007) (xy 101.960537 70.798007) (xy 101.960537 69.681695) (xy 100.766311 69.681695)
+					(xy 100.505086 69.786701) (xy 100.421074 70.022903) (xy 99.265806 70.022903) (xy 99.265806 69.954392)
+					(xy 99.290125 69.676133) (xy 99.385418 69.365367) (xy 99.54676 69.101975) (xy 99.767665 68.892599)
+					(xy 100.041645 68.743879) (xy 100.362211 68.662457) (xy 100.574214 68.64867) (xy 103.115806 68.64867)
+				)
 			)
-			(justify left bottom mirror)
+			(polygon
+				(pts
+					(xy 96.30375 70.196193) (xy 96.57443 70.144322) (xy 96.869797 70.181265) (xy 97.137819 70.322295)
+					(xy 97.339711 70.532269) (xy 97.390509 70.607254) (xy 97.421406 70.607254) (xy 97.497976 70.196193)
+					(xy 98.537718 70.196193) (xy 98.537718 74.065) (xy 97.421406 74.065) (xy 97.421406 71.628189) (xy 97.352014 71.349279)
+					(xy 97.139112 71.15694) (xy 96.905565 71.109661) (xy 96.30375 71.109661)
+				)
+			)
+			(polygon
+				(pts
+					(xy 94.033513 70.996821) (xy 93.782645 71.093709) (xy 93.686933 71.348775) (xy 93.686933 74.065)
+					(xy 92.570621 74.065) (xy 92.570621 71.403852) (xy 92.593909 71.072116) (xy 92.661464 70.79595)
+					(xy 92.802882 70.523564) (xy 93.001292 70.32572) (xy 93.24993 70.195593) (xy 93.542031 70.126355)
+					(xy 93.802459 70.110219) (xy 94.107248 70.136751) (xy 94.387749 70.225556) (xy 94.624959 70.386779)
+					(xy 94.773691 70.572327) (xy 94.804588 70.572327) (xy 94.881158 70.196193) (xy 95.9209 70.196193)
+					(xy 95.9209 74.065) (xy 94.804588 74.065) (xy 94.804588 71.551618) (xy 94.746907 71.270558) (xy 94.566325 71.06842)
+					(xy 94.288747 70.996821)
+				)
+			)
+			(polygon
+				(pts
+					(xy 90.478342 70.122174) (xy 90.757144 70.157824) (xy 91.076199 70.241667) (xy 91.336936 70.366314)
+					(xy 91.583992 70.578351) (xy 91.747177 70.851489) (xy 91.820045 71.112998) (xy 91.843876 71.411912)
+					(xy 91.843876 72.850624) (xy 91.820045 73.14948) (xy 91.747177 73.410837) (xy 91.583992 73.683699)
+					(xy 91.336936 73.895425) (xy 91.076199 74.019837) (xy 90.757144 74.103492) (xy 90.478342 74.139052)
+					(xy 90.164706 74.150973) (xy 89.85127 74.139052) (xy 89.573013 74.103492) (xy 89.255084 74.019837)
+					(xy 88.995755 73.895425) (xy 88.750571 73.683699) (xy 88.589037 73.410837) (xy 88.517082 73.14948)
+					(xy 88.493597 72.850624) (xy 88.493597 71.411912) (xy 88.49803 71.355491) (xy 89.609909 71.355491)
+					(xy 89.609909 72.907044) (xy 89.705118 73.16698) (xy 89.956489 73.265715) (xy 90.37964 73.265715)
+					(xy 90.631012 73.16698) (xy 90.726221 72.907044) (xy 90.726221 71.355491) (xy 90.631012 71.095556)
+					(xy 90.37964 70.996821) (xy 89.956489 70.996821) (xy 89.705118 71.095556) (xy 89.609909 71.355491)
+					(xy 88.49803 71.355491) (xy 88.517082 71.112998) (xy 88.589037 70.851489) (xy 88.750571 70.578351)
+					(xy 88.995755 70.366314) (xy 89.255084 70.241667) (xy 89.573013 70.157824) (xy 89.85127 70.122174)
+					(xy 90.164706 70.110219)
+				)
+			)
+			(polygon
+				(pts
+					(xy 84.014916 70.849054) (xy 86.201866 73.033318) (xy 86.201866 74.065) (xy 82.552023 74.065) (xy 82.552023 73.033318)
+					(xy 84.68524 73.033318) (xy 84.68524 73.002421) (xy 82.991294 71.284295) (xy 82.81691 71.066403)
+					(xy 82.681776 70.806931) (xy 82.608814 70.543846) (xy 82.59098 70.32784) (xy 82.59098 69.958422)
+					(xy 82.615299 69.678833) (xy 82.710592 69.366863) (xy 82.871935 69.102692) (xy 83.09284 68.892869)
+					(xy 83.366819 68.743942) (xy 83.687386 68.662461) (xy 83.899389 68.64867) (xy 84.893457 68.64867)
+					(xy 85.172989 68.673047) (xy 85.484757 68.768541) (xy 85.748641 68.930171) (xy 85.958152 69.151388)
+					(xy 86.106804 69.425643) (xy 86.188109 69.746386) (xy 86.201866 69.958422) (xy 86.201866 70.290226)
+					(xy 85.046598 70.290226) (xy 85.046598 70.028276) (xy 84.939921 69.766316) (xy 84.70136 69.681695)
+					(xy 84.092829 69.681695) (xy 83.841458 69.777744) (xy 83.746249 70.030963) (xy 83.746249 70.286196)
+					(xy 83.800735 70.566905) (xy 83.963902 70.803002) (xy 84.014916 70.853084)
+				)
+			)
+			(polygon
+				(pts
+					(xy 80.887806 68.673052) (xy 81.199776 68.768601) (xy 81.463947 68.930396) (xy 81.67377 69.151951)
+					(xy 81.822697 69.426776) (xy 81.904178 69.748386) (xy 81.917969 69.961109) (xy 81.917969 72.753904)
+					(xy 81.893592 73.034323) (xy 81.798098 73.346893) (xy 81.636467 73.611296) (xy 81.415251 73.821106)
+					(xy 81.140996 73.969896) (xy 80.820253 74.05124) (xy 80.608217 74.065) (xy 79.415334 74.065) (xy 79.135745 74.040675)
+					(xy 78.823775 73.945328) (xy 78.559604 73.78382) (xy 78.349781 73.562577) (xy 78.200854 73.288027)
+					(xy 78.119373 72.966594) (xy 78.105582 72.753904) (xy 78.105582 70.030963) (xy 79.260851 70.030963)
+					(xy 79.260851 72.68405) (xy 79.35606 72.937269) (xy 79.607431 73.033318) (xy 80.41612 73.033318)
+					(xy 80.667491 72.937269) (xy 80.7627 72.68405) (xy 80.7627 70.030963) (xy 80.667491 69.777744)
+					(xy 80.41612 69.681695) (xy 79.607431 69.681695) (xy 79.35606 69.777744) (xy 79.260851 70.030963)
+					(xy 78.105582 70.030963) (xy 78.105582 69.961109) (xy 78.129959 69.680633) (xy 78.225453 69.367861)
+					(xy 78.387083 69.10317) (xy 78.6083 68.893049) (xy 78.882555 68.743984) (xy 79.203298 68.662463)
+					(xy 79.415334 68.64867) (xy 80.608217 68.64867)
+				)
+			)
+			(polygon
+				(pts
+					(xy 75.283234 70.849054) (xy 77.470184 73.033318) (xy 77.470184 74.065) (xy 73.820341 74.065) (xy 73.820341 73.033318)
+					(xy 75.953558 73.033318) (xy 75.953558 73.002421) (xy 74.259612 71.284295) (xy 74.085229 71.066403)
+					(xy 73.950095 70.806931) (xy 73.877132 70.543846) (xy 73.859298 70.32784) (xy 73.859298 69.958422)
+					(xy 73.883617 69.678833) (xy 73.97891 69.366863) (xy 74.140253 69.102692) (xy 74.361158 68.892869)
+					(xy 74.635137 68.743942) (xy 74.955704 68.662461) (xy 75.167707 68.64867) (xy 76.161775 68.64867)
+					(xy 76.441307 68.673047) (xy 76.753076 68.768541) (xy 77.016959 68.930171) (xy 77.226471 69.151388)
+					(xy 77.375122 69.425643) (xy 77.456427 69.746386) (xy 77.470184 69.958422) (xy 77.470184 70.290226)
+					(xy 76.314916 70.290226) (xy 76.314916 70.028276) (xy 76.208239 69.766316) (xy 75.969678 69.681695)
+					(xy 75.361147 69.681695) (xy 75.109776 69.777744) (xy 75.014567 70.030963) (xy 75.014567 70.286196)
+					(xy 75.069053 70.566905) (xy 75.232221 70.803002) (xy 75.283234 70.853084)
+				)
+			)
+			(polygon
+				(pts
+					(xy 73.493911 72.173583) (xy 73.493911 73.205265) (xy 70.922766 73.205265) (xy 70.922766 74.065)
+					(xy 69.767498 74.065) (xy 69.767498 73.205265) (xy 69.074337 73.205265) (xy 69.074337 72.173583)
+					(xy 69.767498 72.173583) (xy 70.922766 72.173583) (xy 72.323866 72.173583) (xy 72.323866 72.142686)
+					(xy 70.96038 70.196193) (xy 70.922766 70.196193) (xy 70.922766 72.173583) (xy 69.767498 72.173583)
+					(xy 69.767498 68.64867) (xy 71.05307 68.64867)
+				)
+			)
 		)
 	)
